File: sr_lights/sr_lights.sch (EAGLE design)
At the start: 33 parts, among them T1 BC847, T2 BC847, T3 BC847, T4 BC847, T5 BC847, T6 BC847, T7 BC847, T8 BC847

Commit message: Added reverse current protection for external power, added version text
Parts:
- added Q1: IRLML2244TRPbF, we-transistor:MOSFET-P-SOT23
Connections:
- new net VCC2_RAW: EXT_PWR_IN.1, Q1.D
- net GND: now also Q1.G
- net VCC2: now also Q1.S; no longer EXT_PWR_IN.1
Other:
- note added: "REVERSE PWR PROTECTION"
Changed lines of the file:
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@@
 <grid distance="0.1" unitdist="inch" unit="inch" style="lines" multiple="1" display="no" altdistance="0.01" altunitdist="inch" altunit="inch"/>
 <layers>
-<layer number="1" name="Top" color="4" fill="1" visible="yes" active="no"/>
-<layer number="16" name="Bottom" color="1" fill="1" visible="yes" active="no"/>
-<layer number="17" name="Pads" color="2" fill="1" visible="yes" active="no"/>
-<layer number="18" name="Vias" color="2" fill="1" visible="yes" active="no"/>
-<layer number="19" name="Unrouted" color="6" fill="1" visible="yes" active="no"/>
-<layer number="20" name="Dimension" color="15" fill="1" visible="yes" active="no"/>
-<layer number="21" name="tPlace" color="7" fill="1" visible="yes" active="no"/>
-<layer number="22" name="bPlace" color="7" fill="1" visible="yes" active="no"/>
-<layer number="23" name="tOrigins" color="15" fill="1" visible="yes" active="no"/>
-<layer number="24" name="bOrigins" color="15" fill="1" visible="yes" active="no"/>
-<layer number="25" name="tNames" color="7" fill="1" visible="yes" active="no"/>
-<layer number="26" name="bNames" color="7" fill="1" visible="yes" active="no"/>
-<layer number="27" name="tValues" color="7" fill="1" visible="yes" active="no"/>
-<layer number="28" name="bValues" color="7" fill="1" visible="yes" active="no"/>
+<layer number="1" name="Top" color="4" fill="1" visible="no" active="no"/>
+<layer number="16" name="Bottom" color="1" fill="1" visible="no" active="no"/>
+<layer number="17" name="Pads" color="2" fill="1" visible="no" active="no"/>
+<layer number="18" name="Vias" color="2" fill="1" visible="no" active="no"/>
+<layer number="19" name="Unrouted" color="6" fill="1" visible="no" active="no"/>
+<layer number="20" name="Dimension" color="15" fill="1" visible="no" active="no"/>
+<layer number="21" name="tPlace" color="7" fill="1" visible="no" active="no"/>
+<layer number="22" name="bPlace" color="7" fill="1" visible="no" active="no"/>
+<layer number="23" name="tOrigins" color="15" fill="1" visible="no" active="no"/>
+<layer number="24" name="bOrigins" color="15" fill="1" visible="no" active="no"/>
+<layer number="25" name="tNames" color="7" fill="1" visible="no" active="no"/>
+<layer number="26" name="bNames" color="7" fill="1" visible="no" active="no"/>
+<layer number="27" name="tValues" color="7" fill="1" visible="no" active="no"/>
+<layer number="28" name="bValues" color="7" fill="1" visible="no" active="no"/>
 <layer number="29" name="tStop" color="7" fill="3" visible="no" active="no"/>
 <layer number="30" name="bStop" color="7" fill="6" visible="no" active="no"/>
@@
 <layer number="35" name="tGlue" color="7" fill="4" visible="no" active="no"/>
 <layer number="36" name="bGlue" color="7" fill="5" visible="no" active="no"/>
-<layer number="37" name="tTest" color="7" fill="1" visible="yes" active="no"/>
-<layer number="38" name="bTest" color="7" fill="1" visible="yes" active="no"/>
+<layer number="37" name="tTest" color="7" fill="1" visible="no" active="no"/>
+<layer number="38" name="bTest" color="7" fill="1" visible="no" active="no"/>
 <layer number="39" name="tKeepout" color="4" fill="11" visible="no" active="no"/>
 <layer number="40" name="bKeepout" color="1" fill="11" visible="no" active="no"/>
@@
 <layer number="44" name="Drills" color="7" fill="1" visible="no" active="no"/>
 <layer number="45" name="Holes" color="7" fill="1" visible="no" active="no"/>
-<layer number="46" name="Milling" color="3" fill="1" visible="yes" active="no"/>
-<layer number="47" name="Measures" color="7" fill="1" visible="yes" active="no"/>
-<layer number="48" name="Document" color="7" fill="1" visible="yes" active="no"/>
-<layer number="49" name="Reference" color="7" fill="1" visible="yes" active="no"/>
-<layer number="51" name="tDocu" color="7" fill="1" visible="yes" active="no"/>
-<layer number="52" name="bDocu" color="7" fill="1" visible="yes" active="no"/>
+<layer number="46" name="Milling" color="3" fill="1" visible="no" active="no"/>
+<layer number="47" name="Measures" color="7" fill="1" visible="no" active="no"/>
+<layer number="48" name="Document" color="7" fill="1" visible="no" active="no"/>
+<layer number="49" name="Reference" color="7" fill="1" visible="no" active="no"/>
+<layer number="51" name="tDocu" color="7" fill="1" visible="no" active="no"/>
+<layer number="52" name="bDocu" color="7" fill="1" visible="no" active="no"/>
 <layer number="90" name="Modules" color="5" fill="1" visible="yes" active="yes"/>
 <layer number="91" name="Nets" color="2" fill="1" visible="yes" active="yes"/>
@@
 </part>
 <part name="C2" library="eagle-ltspice" deviceset="C" device="" value="100nF"/>
+<part name="Q1" library="we-transistor" deviceset="MOSFET-P" device="-SOT23" value="IRLML2244TRPbF"/>
 </parts>
 <sheets>
@@
 <wire x1="182.88" y1="71.12" x2="182.88" y2="0" width="0.1524" layer="97" style="shortdash"/>
 <wire x1="182.88" y1="0" x2="231.14" y2="0" width="0.1524" layer="97" style="shortdash"/>
-<wire x1="231.14" y1="0" x2="231.14" y2="71.12" width="0.1524" layer="97" style="shortdash"/>
 <wire x1="231.14" y1="71.12" x2="182.88" y2="71.12" width="0.1524" layer="97" style="shortdash"/>
 <text x="228.6" y="73.66" size="1.778" layer="97" rot="R180">POWER</text>
@@
 <text x="2.54" y="157.48" size="1.778" layer="97" rot="MR180">LIGHT_SITCHES</text>
 <text x="71.12" y="83.82" size="1.778" layer="97" rot="R180">LIGHTS_CON</text>
+<wire x1="231.14" y1="71.12" x2="231.14" y2="0" width="0.1524" layer="97" style="shortdash"/>
+<wire x1="231.14" y1="0" x2="256.54" y2="0" width="0.1524" layer="97" style="shortdash"/>
+<wire x1="256.54" y1="0" x2="256.54" y2="71.12" width="0.1524" layer="97" style="shortdash"/>
+<wire x1="256.54" y1="71.12" x2="231.14" y2="71.12" width="0.1524" layer="97" style="shortdash"/>
+<text x="254" y="76.2" size="1.778" layer="97" rot="R180">REVERSE PWR
+PROTECTION</text>
 </plain>
 <instances>
@@
 </instance>
 <instance part="C2" gate="G$1" x="210.82" y="45.72"/>
+<instance part="Q1" gate="T" x="243.84" y="38.1"/>
 </instances>
 <busses>
@@
 </segment>
 </bus>
-<bus name="OUTS:LI[0..7],VCC1,VCC2,GND">
+<bus name="OUTS:LI[0..7],VCC1,VCC2,GND,VCC2_RAW">
 <segment>
 <wire x1="5.08" y1="132.08" x2="5.08" y2="73.66" width="0.762" layer="92"/>
@@
 <wire x1="5.08" y1="73.66" x2="73.66" y2="73.66" width="0.762" layer="92"/>
 <wire x1="190.5" y1="5.08" x2="190.5" y2="66.04" width="0.762" layer="92"/>
+<wire x1="190.5" y1="5.08" x2="231.14" y2="5.08" width="0.762" layer="92"/>
+<wire x1="231.14" y1="5.08" x2="231.14" y2="66.04" width="0.762" layer="92"/>
 </segment>
 </bus>
@@
 <pinref part="EXT_PWR_IN" gate="G$1" pin="2"/>
 <wire x1="116.84" y1="17.78" x2="116.84" y2="5.08" width="0.1524" layer="91"/>
+<label x="116.84" y="7.62" size="1.778" layer="95"/>
 </segment>
 <segment>
 <pinref part="EXT_PWR_OUT" gate="G$1" pin="2"/>
 <wire x1="165.1" y1="17.78" x2="165.1" y2="5.08" width="0.1524" layer="91"/>
+<label x="165.1" y="7.62" size="1.778" layer="95"/>
 </segment>
 <segment>
@@
 <wire x1="93.98" y1="63.5" x2="111.76" y2="63.5" width="0.1524" layer="91"/>
 <wire x1="93.98" y1="5.08" x2="93.98" y2="63.5" width="0.1524" layer="91"/>
-<label x="93.98" y="7.62" size="1.778" layer="95" rot="MR0"/>
+<label x="93.98" y="12.7" size="1.778" layer="95" rot="MR0"/>
 </segment>
 <segment>
@@
 <wire x1="198.12" y1="15.24" x2="198.12" y2="17.78" width="0.1524" layer="91"/>
 <label x="193.04" y="12.7" size="1.778" layer="95"/>
+</segment>
+<segment>
+<pinref part="Q1" gate="T" pin="G"/>
+<wire x1="238.76" y1="35.56" x2="231.14" y2="35.56" width="0.1524" layer="91"/>
+<label x="233.68" y="35.56" size="1.778" layer="95"/>
 </segment>
 </net>
@@
 </segment>
 <segment>
-<pinref part="EXT_PWR_IN" gate="G$1" pin="1"/>
-<wire x1="114.3" y1="17.78" x2="114.3" y2="5.08" width="0.1524" layer="91"/>
-</segment>
-<segment>
 <pinref part="EXT_PWR_OUT" gate="G$1" pin="1"/>
 <wire x1="162.56" y1="17.78" x2="162.56" y2="5.08" width="0.1524" layer="91"/>
+<label x="162.56" y="7.62" size="1.778" layer="95" rot="MR0"/>
 </segment>
 <segment>
@@
 <label x="193.04" y="27.94" size="1.778" layer="95"/>
 </segment>
+<segment>
+<pinref part="Q1" gate="T" pin="S"/>
+<wire x1="243.84" y1="33.02" x2="243.84" y2="30.48" width="0.1524" layer="91"/>
+<wire x1="231.14" y1="30.48" x2="243.84" y2="30.48" width="0.1524" layer="91"/>
+<label x="233.68" y="30.48" size="1.778" layer="95"/>
+</segment>
 </net>
 <net name="VCC1" class="2">
@@
 <wire x1="109.22" y1="55.88" x2="109.22" y2="60.96" width="0.1524" layer="91"/>
 <wire x1="96.52" y1="60.96" x2="109.22" y2="60.96" width="0.1524" layer="91"/>
-<label x="96.52" y="7.62" size="1.778" layer="95"/>
+<label x="96.52" y="12.7" size="1.778" layer="95"/>
 </segment>
 <segment>
@@
 </segment>
 </net>
+<net name="VCC2_RAW" class="0">
+<segment>
+<pinref part="Q1" gate="T" pin="D"/>
+<wire x1="243.84" y1="43.18" x2="231.14" y2="43.18" width="0.1524" layer="91"/>
+<label x="233.68" y="43.18" size="1.778" layer="95"/>
+</segment>
+<segment>
+<pinref part="EXT_PWR_IN" gate="G$1" pin="1"/>
+<wire x1="114.3" y1="17.78" x2="114.3" y2="5.08" width="0.1524" layer="91"/>
+<label x="114.3" y="7.62" size="1.778" layer="95" rot="MR0"/>
+</segment>
+</net>
 </nets>
 </sheet>
@@
 </schematic>
 </drawing>
+<compatibility>
+<note version="6.3" minversion="6.2.2" severity="warning">
+Since Version 6.2.2 text objects can contain more than one line,
+which will not be processed correctly with this version.
+</note>
+</compatibility>
 </eagle>
